File: Circuit/Circuit.kicad_pcb (KiCad board)
At the start: 2 copper layers, 80 x 80 mm, 20 parts, among them J1 M5Stamp_Pico, J10 PinHeader, J2 Conn_01x02_Pin, J3 VL53L4CX, J4 A295-CTRPB-1, J5 Conn_01x12_Pin, J6 Conn_01x02_Pin, J7 Conn_01x03_Pin, J8 Conn_01x03_Pin, J9 PinHeader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

Commit message: Update to support M5stamp footprint correction
Parts:
- moved J10 2.56 mm to (178.1, 71.5)
- moved J9 2.50 mm to (178.1, 63.2)
- moved J1 1.34 mm to (192.0, 57.5)
Routing:
- net Net-(J1-Pin_12): track 27.1 -> 24.4 mm
- net +3V3: track 148.2 -> 149.0 mm
Other:
- board text removed: "G"
